Commit message: Add docking camera frames to robot description
Give the docking camera a real place in the TF tree so RViz/Nav2 can locate
detections and a Gazebo camera can be mounted later.

- amr_description: add camera_link (front mount) and camera_optical_frame
  (REP-103 optical convention) to the xacro, matching the frame_id used by
  amr_vision and the controller's camera_forward_offset.
- Note the Gazebo camera sensor as the follow-up in the docking guide.

Co-Authored-By: Claude Opus 4.8 <noreply@anthropic.com>
Claude-Session: https://claude.ai/code/session_01MEj8QSrWSni8uVEuK3MqyA

File: src/amr_description/urdf/amr_demo_robot.urdf.xacro (robot description, xacro)
@@ -91,3 +91,25 @@
     <origin xyz="0.23 0 0.175" rpy="0 0 0"/>
   </joint>
+  <!-- Forward-facing docking camera. camera_link is the mounting frame;
+       camera_optical_frame follows the REP-103 optical convention
+       (x right, y down, z forward) used by amr_vision. -->
+  <link name="camera_link">
+    <visual>
+      <geometry>
+        <box size="0.03 0.09 0.03"/>
+      </geometry>
+      <material name="lidar_black"/>
+    </visual>
+  </link>
+  <joint name="camera_joint" type="fixed">
+    <parent link="base_link"/>
+    <child link="camera_link"/>
+    <origin xyz="0.40 0 0.10" rpy="0 0 0"/>
+  </joint>
+  <link name="camera_optical_frame"/>
+  <joint name="camera_optical_joint" type="fixed">
+    <parent link="camera_link"/>
+    <child link="camera_optical_frame"/>
+    <origin xyz="0 0 0" rpy="-1.57079632679 0 -1.57079632679"/>
+  </joint>
 </robot>
